Commit message: feat: change wrist_ft_sensor_frame_joint to fixed joint and implement FT sensor wrench computation

File: data/urdf/hsrb4s.urdf (robot description, URDF)
Before this commit: robot hsrb, 48 links, 47 joints
Joints:
- joint wrist_ft_sensor_frame_joint: limit lower=0 upper=0 effort=100.0 velocity=1.5 -> (none); type revolute -> fixed
